File: hardware/RegulatedPowerSupply3.3V5V/RegulatedPowerSupply3.3V5V.kicad_sch (KiCad schematic)
At the start: 12 parts, among them J1 1x04 PIN

Commit message: KiCad
Parts:
- PWROFF_IND1: renamed from PWROFF_IND; footprint (none) -> Connector_PinHeader_2.54mm:PinHeader_1x02_P2.54mm_Vertical
- renumbered 1x02_PIN to AMS1117_VINGND1, 1x02_PIN to AMS1117_VOUTGND1, J1 to POWER_RAIL1
Connections:
- net TP4056+: now reaches MT3608_Module1.1 (VIN+), OnOff_SlidingSW1.2 (C)
- net TP4056+: now also OnOff_SlidingSW1.1 (B), TP4056_Module1.3 (OUT+)
- net at OnOff_SlidingSW1.3 (A), PWROFF_IND1.1 (Pin_1): no longer names the net of OnOff_SlidingSW1.3 (A), PWROFF_IND1.1 (Pin_1)
Changed lines of the file:
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@@
-	)
-	(junction
-		(at 97.79 44.45)
-		(diameter 0)
-		(color 0 0 0 0)
-	)
-	(junction
-		(at 116.84 105.41)
-		(diameter 0)
-		(color 0 0 0 0)
 	)
 	(junction
@@
 	)
 	(junction
+		(at 96.52 105.41)
+		(diameter 0)
+		(color 0 0 0 0)
+	)
+	(junction
 		(at 63.5 63.5)
 		(diameter 0)
@@
 	)
 	(junction
+		(at 95.25 44.45)
+		(diameter 0)
+		(color 0 0 0 0)
+	)
+	(junction
 		(at 127 97.79)
 		(diameter 0)
@@
 	(wire
 		(pts
-			(xy 97.79 44.45) (xy 113.03 44.45)
-		)
-		(stroke
-			(width 0)
-			(type default)
-		)
-	)
-	(wire
-		(pts
-			(xy 72.39 44.45) (xy 97.79 44.45)
+			(xy 72.39 44.45) (xy 95.25 44.45)
 		)
 		(stroke
@@
 	(wire
 		(pts
+			(xy 96.52 105.41) (xy 127 105.41)
+		)
+		(stroke
+			(width 0)
+			(type default)
+		)
+	)
+	(wire
+		(pts
 			(xy 166.37 129.54) (xy 166.37 113.03)
 		)
@@
 	(wire
 		(pts
+			(xy 93.98 54.61) (xy 93.98 55.88)
+		)
+		(stroke
+			(width 0)
+			(type default)
+		)
+	)
+	(wire
+		(pts
 			(xy 105.41 58.42) (xy 105.41 73.66)
 		)
@@
 	(wire
 		(pts
-			(xy 116.84 105.41) (xy 116.84 106.68)
+			(xy 88.9 97.79) (xy 88.9 105.41)
+		)
+		(stroke
+			(width 0)
+			(type default)
+		)
+	)
+	(wire
+		(pts
+			(xy 96.52 105.41) (xy 96.52 107.95)
+		)
+		(stroke
+			(width 0)
+			(type default)
+		)
+	)
+	(wire
+		(pts
+			(xy 88.9 97.79) (xy 92.71 97.79)
+		)
+		(stroke
+			(width 0)
+			(type default)
+		)
+	)
+	(wire
+		(pts
+			(xy 93.98 55.88) (xy 88.9 55.88)
 		)
 		(stroke
@@
 	(wire
 		(pts
-			(xy 87.63 97.79) (xy 87.63 105.41)
-		)
-		(stroke
-			(width 0)
-			(type default)
-		)
-	)
-	(wire
-		(pts
 			(xy 139.7 80.01) (xy 134.62 80.01)
 		)
@@
 	(wire
 		(pts
+			(xy 123.19 76.2) (xy 123.19 92.71)
+		)
+		(stroke
+			(width 0)
+			(type default)
+		)
+	)
+	(wire
+		(pts
 			(xy 57.15 101.6) (xy 57.15 102.87)
 		)
@@
 	(wire
 		(pts
-			(xy 87.63 105.41) (xy 116.84 105.41)
+			(xy 88.9 105.41) (xy 96.52 105.41)
 		)
 		(stroke
@@
 	(wire
 		(pts
+			(xy 95.25 44.45) (xy 95.25 54.61)
+		)
+		(stroke
+			(width 0)
+			(type default)
+		)
+	)
+	(wire
+		(pts
 			(xy 113.03 44.45) (xy 113.03 46.99)
 		)
@@
 	(wire
 		(pts
-			(xy 127 105.41) (xy 116.84 105.41)
-		)
-		(stroke
-			(width 0)
-			(type default)
-		)
-	)
-	(wire
-		(pts
 			(xy 68.58 73.66) (xy 105.41 73.66)
 		)
@@
 	(wire
 		(pts
-			(xy 87.63 97.79) (xy 92.71 97.79)
-		)
-		(stroke
-			(width 0)
-			(type default)
-		)
-	)
-	(wire
-		(pts
 			(xy 50.8 82.55) (xy 63.5 82.55)
 		)
@@
 	(wire
 		(pts
-			(xy 123.19 76.2) (xy 123.19 92.71)
-		)
-		(stroke
-			(width 0)
-			(type default)
-		)
-	)
-	(wire
-		(pts
 			(xy 92.71 124.46) (xy 92.71 137.16)
 		)
@@
 	(wire
 		(pts
-			(xy 88.9 55.88) (xy 97.79 55.88)
+			(xy 93.98 54.61) (xy 95.25 54.61)
 		)
 		(stroke
@@
 	(wire
 		(pts
+			(xy 95.25 44.45) (xy 113.03 44.45)
+		)
+		(stroke
+			(width 0)
+			(type default)
+		)
+	)
+	(wire
+		(pts
 			(xy 127 90.17) (xy 137.16 90.17)
 		)
@@
 		)
 	)
-	(wire
-		(pts
-			(xy 97.79 44.45) (xy 97.79 55.88)
-		)
-		(stroke
-			(width 0)
-			(type default)
+	(label "TP4056+"
+		(at 123.19 86.36 0)
+		(effects
+			(font
+				(size 1.27 1.27)
+			)
+			(justify left bottom)
 		)
 	)
@@
 	)
 	(label "BATT+"
-		(at 54.61 87.63 0)
+		(at 52.07 87.63 0)
 		(effects
 			(font
@@
 		)
 	)
-	(label ""
-		(at 124.46 68.58 0)
+	(label "TP4056+"
+		(at 134.62 83.82 0)
 		(effects
 			(font
@@
 	)
 	(label "3.3V"
-		(at 55.88 82.55 0)
+		(at 52.07 82.55 0)
 		(effects
 			(font
@@
 	)
 	(label "5V"
-		(at 55.88 85.09 0)
+		(at 52.07 85.09 0)
 		(effects
 			(font
@@
 		(dnp no)
 		(fields_autoplaced yes)
-		(property "Reference" "J1"
+		(property "Reference" "POWER_RAIL1"
 			(at 46.355 77.47 0)
 			(effects
@@
 			(project ""
 				(path "/171bd10b-7e6c-47c5-ae33-4e3750b9f549"
-					(reference "J1")
+					(reference "POWER_RAIL1")
 					(unit 1)
 				)
@@
 		(on_board yes)
 		(dnp no)
-		(property "Reference" "1x02_PIN"
-			(at 88.138 52.832 0)
+		(property "Reference" "AMS1117_VINGND1"
+			(at 85.598 51.562 0)
 			(effects
 				(font
@@
 			(project ""
 				(path "/171bd10b-7e6c-47c5-ae33-4e3750b9f549"
-					(reference "1x02_PIN")
+					(reference "AMS1117_VINGND1")
 					(unit 1)
 				)
@@
 		(on_board yes)
 		(dnp no)
-		(property "Reference" "1x02_PIN"
-			(at 74.93 52.07 0)
+		(property "Reference" "AMS1117_VOUTGND1"
+			(at 74.422 48.514 0)
 			(effects
 				(font
@@
 			(project ""
 				(path "/171bd10b-7e6c-47c5-ae33-4e3750b9f549"
-					(reference "1x02_PIN")
+					(reference "AMS1117_VOUTGND1")
 					(unit 1)
 				)
@@
 	(symbol
 		(lib_id "power:GND")
-		(at 116.84 106.68 0)
+		(at 96.52 107.95 0)
 		(unit 1)
 		(exclude_from_sim no)
@@
 		(fields_autoplaced yes)
 		(property "Reference" "#PWR03"
-			(at 116.84 113.03 0)
+			(at 96.52 114.3 0)
 			(effects
 				(font
@@
 		)
 		(property "Value" "GND"
-			(at 116.84 111.76 0)
+			(at 96.52 113.03 0)
 			(effects
 				(font
@@
 		)
 		(property "Footprint" ""
-			(at 116.84 106.68 0)
+			(at 96.52 107.95 0)
 			(effects
 				(font
@@
 		)
 		(property "Datasheet" ""
-			(at 116.84 106.68 0)
+			(at 96.52 107.95 0)
 			(effects
 				(font
@@
 		)
 		(property "Description" "Power symbol creates a global label with name \"GND\" , ground"
-			(at 116.84 106.68 0)
+			(at 96.52 107.95 0)
 			(effects
 				(font
@@
 		(on_board yes)
 		(dnp no)
-		(fields_autoplaced yes)
-		(property "Reference" "PWROFF_IND"
-			(at 117.475 63.5 0)
+		(property "Reference" "PWROFF_IND1"
+			(at 115.062 65.024 0)
 			(effects
 				(font
@@
 			)
 		)
-		(property "Footprint" ""
+		(property "Footprint" "Connector_PinHeader_2.54mm:PinHeader_1x02_P2.54mm_Vertical"
 			(at 116.84 68.58 0)
 			(effects
@@
 			(project ""
 				(path "/171bd10b-7e6c-47c5-ae33-4e3750b9f549"
-					(reference "PWROFF_IND")
+					(reference "PWROFF_IND1")
 					(unit 1)
 				)
