File: hardware/PhysicalButtons/PhysicalButtons.kicad_sch (KiCad schematic)
At the start: 24 parts

Commit message: KiCad
Parts:
- added Battery: Conn_01x02_Pin, symbol Connector:Conn_01x02_Pin
- added C3, C4, C5: 0.1uF, Capacitor_THT:C_Disc_D5.0mm_W2.5mm_P2.50mm, symbol Device:C
Connections:
- net EC11_PHA: now also C4.1
- net EC11_PHB: now also C3.1
- net GND: now also C3.2, C4.2, C5.2
- net MCPCLK: now also ESP32-S3_MC1.15 (GPIO9/ADC1_CH8), R6.2; no longer ESP32-S3_MC1.12 (GPIO8/ADC1_CH7), R5.2
- net MCPDATA: now also ESP32-S3_MC1.12 (GPIO8/ADC1_CH7), R5.2; no longer ESP32-S3_MC1.15 (GPIO9/ADC1_CH8), R6.2
- net at C1.2, C2.1, ESP32-S3_MC1.1 (3V3)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: now also C5.1
- net at ESP32-S3_MC1.13 (GPIO3/ADC1_CH2): now also Battery.1 (Pin_1)
Other:
- moved on the sheet: C1, C2, E6B2_ROTARYENC1, ESP32-S3_MC1, I/O_EX1, JOY_SOCK1, LOCK_PANEL_TOGGLE1, MOBJECTIVE_SELECT1, PAIR1, R1, R2, R3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
