File: hardware/PhysicalButtons/_autosave-PhysicalButtons.kicad_pcb (KiCad board)
At the start: 2 copper layers, 177.2 x 98.8 mm, 20 parts

Commit message: KiCad
Parts:
- added C2: 0.1uF, Capacitor_THT:C_Disc_D5.0mm_W2.5mm_P2.50mm, F.Cu at (57.7, 148.4)
- added C3: 0.1uF, Capacitor_THT:C_Disc_D5.0mm_W2.5mm_P2.50mm, F.Cu at (57.7, 152.5)
- added C4: 0.1uF, Capacitor_THT:C_Disc_D5.0mm_W2.5mm_P2.50mm, F.Cu at (57.7, 156.5)
- added C5: 0.1uF, Capacitor_THT:C_Disc_D5.0mm_W2.5mm_P2.50mm, F.Cu at (57.7, 160.6)
- added R4: 10k, Resistor_THT:R_Axial_DIN0411_L9.9mm_D3.6mm_P12.70mm_Horizontal, F.Cu at (64.2, 149.0)
- added R5: 4.7k, Resistor_THT:R_Axial_DIN0207_L6.3mm_D2.5mm_P7.62mm_Horizontal, F.Cu at (63.8, 158.7)
- added R6: 4.7k, Resistor_THT:R_Axial_DIN0207_L6.3mm_D2.5mm_P7.62mm_Horizontal, F.Cu at (63.8, 162.8)
- added R7: 10k, Resistor_THT:R_Axial_DIN0411_L9.9mm_D3.6mm_P12.70mm_Horizontal, F.Cu at (64.2, 154.1)
- moved E6B2_ROTARYENC1 101.2 mm to (133.4, 162.3)
- moved ST7789_DISP1 67.8 mm to (27.5, 68.6)
- moved MOBJECTIVE_SELECT1 36.2 mm to (203.3, 118.7)
- moved SAVE_CURR_POS1 36.2 mm to (184.3, 77.3)
- moved UNASSIGNED2 36.2 mm to (241.3, 101.7)
- moved SLEEP1 36.2 mm to (123.3, 58.6)
- moved VIN3.3VGND1 36.2 mm to (102.4, 41.7)
- moved C1 36.2 mm to (201.1, 90.8)
- moved JOY_SOCK1 36.2 mm to (114.4, 86.6)
- moved LOCK_PANEL_TOGGLE1 36.2 mm to (194.3, 63.9)
- moved R1 36.2 mm to (216.2, 93.4)
- moved R2 36.2 mm to (103.4, 146.0)
- moved R3 36.2 mm to (103.4, 151.1)
- moved RESET_POS1 36.2 mm to (167.3, 76.9)
- moved TO_ESP32MC1 36.2 mm to (192.4, 102.8)
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Connections:
- net /FINECOARSE_SWITCH renamed /JOY_SW
- ESP32-S3_MC1 pad 12: /MCPCLK -> /MCPDATA
- ESP32-S3_MC1 pad 13: /E6B2_PHZ -> unconnected-(ESP32-S3_MC1-GPIO3/ADC1_CH2-Pad13)
- ESP32-S3_MC1 pad 15: /MCPDATA -> /MCPCLK
- ESP32-S3_MC1 pad 4: unconnected-(ESP32-S3_MC1-GPIO4/ADC1_CH3-Pad4) -> /E6B2_PHZ
- ESP32-S3_MC1 pad 40: /E6B2_PHB -> /JOY_VRy
- ESP32-S3_MC1 pad 41: /E6B2_PHA -> /JOY_VRx
- ESP32-S3_MC1 pad 5: unconnected-(ESP32-S3_MC1-GPIO5/ADC1_CH4-Pad5) -> /E6B2_PHB
- ESP32-S3_MC1 pad 6: unconnected-(ESP32-S3_MC1-GPIO6/ADC1_CH5-Pad6) -> /E6B2_PHA
